File: PCB/fietscomputer_mainboard_ESP32/fietscomputer_mainboard_ESP32-2.kicad_sch (KiCad schematic)
At the start: 25 parts, among them J1 USB_C_Receptacle_USB2.0_14P, J2 Conn_01x04_Pin, SW1 RESET1, SW2 BOOT1, SW4 PAGE_BUTTON, SW5 LAP_BUTTON, SW6 MAIN_BUTTON, SW7 ZOOM-_BUTTON, SW8 ZOOM+_BUTTON, U1 ESP32-S3-WROOM-1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

Commit message: new main
Parts:
- removed J2: Conn_01x04_Pin, Connector_PinHeader_2.54mm:PinHeader_1x04_P2.54mm_Vertical, symbol Connector:Conn_01x04_Pin
Other:
- note removed: "SCREEN"
